File: EnvFollowerSim/EnvFollowerSim.kicad_sch (KiCad schematic)
At the start: 21 parts, among them U1 TL074

Commit message: env detector sim tweaks
Parts:
- R2: value 22k -> 10k
- R6: value 47k -> 100k
Connections:
- net EnvCap: now also U1.12 (+)
- net FullRect: now also D3.1 (K), R10.1; no longer D3.2 (A), U1.8
- net vEnv: now reaches U1.13 (-)
- net vEnv: now also U1.14
- new net: D3.2 (A), U1.8
Other:
- moved on the sheet: U1D
Changed lines of the file:
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@@
 	)
 	(junction
+		(at 193.294 52.07)
+		(diameter 0)
+		(color 0 0 0 0)
+	)
+	(junction
 		(at 57.15 70.612)
 		(diameter 0)
@@
 	)
 	(junction
-		(at 161.544 55.88)
+		(at 210.566 58.166)
 		(diameter 0)
 		(color 0 0 0 0)
 	)
 	(junction
-		(at 210.566 58.166)
+		(at 42.672 57.15)
 		(diameter 0)
 		(color 0 0 0 0)
 	)
 	(junction
-		(at 42.672 57.15)
+		(at 173.736 55.88)
 		(diameter 0)
 		(color 0 0 0 0)
@@
 	(wire
 		(pts
+			(xy 218.44 39.624) (xy 214.884 39.624)
+		)
+		(stroke
+			(width 0)
+			(type default)
+		)
+	)
+	(wire
+		(pts
+			(xy 214.884 39.624) (xy 214.884 50.038)
+		)
+		(stroke
+			(width 0)
+			(type default)
+		)
+	)
+	(wire
+		(pts
 			(xy 193.294 68.58) (xy 193.294 69.85)
 		)
@@
 	(wire
 		(pts
+			(xy 173.736 41.91) (xy 173.736 55.88)
+		)
+		(stroke
+			(width 0)
+			(type default)
+		)
+	)
+	(wire
+		(pts
 			(xy 57.15 62.23) (xy 59.436 62.23)
 		)
@@
 	(wire
 		(pts
+			(xy 236.982 37.084) (xy 233.68 37.084)
+		)
+		(stroke
+			(width 0)
+			(type default)
+		)
+	)
+	(wire
+		(pts
 			(xy 119.888 68.834) (xy 127.254 68.834)
 		)
@@
 	(wire
 		(pts
+			(xy 173.736 55.88) (xy 176.022 55.88)
+		)
+		(stroke
+			(width 0)
+			(type default)
+		)
+	)
+	(wire
+		(pts
 			(xy 57.15 72.644) (xy 57.15 70.612)
 		)
@@
 	(wire
 		(pts
+			(xy 236.982 50.038) (xy 236.982 37.084)
+		)
+		(stroke
+			(width 0)
+			(type default)
+		)
+	)
+	(wire
+		(pts
 			(xy 127.254 68.834) (xy 127.254 67.31)
 		)
@@
 	(wire
 		(pts
-			(xy 161.544 55.88) (xy 161.544 41.91)
+			(xy 23.622 57.15) (xy 23.622 60.96)
 		)
 		(stroke
@@
 	(wire
 		(pts
-			(xy 23.622 57.15) (xy 23.622 60.96)
+			(xy 142.24 58.42) (xy 137.414 58.42)
 		)
 		(stroke
@@
 	(wire
 		(pts
-			(xy 142.24 58.42) (xy 137.414 58.42)
+			(xy 193.294 34.544) (xy 193.294 52.07)
 		)
 		(stroke
@@
 	(wire
 		(pts
-			(xy 161.544 41.91) (xy 155.448 41.91)
+			(xy 155.448 41.91) (xy 173.736 41.91)
 		)
 		(stroke
@@
 	(wire
 		(pts
-			(xy 161.544 55.88) (xy 164.084 55.88)
+			(xy 157.48 55.88) (xy 164.084 55.88)
 		)
 		(stroke
@@
 	(wire
 		(pts
+			(xy 214.884 50.038) (xy 236.982 50.038)
+		)
+		(stroke
+			(width 0)
+			(type default)
+		)
+	)
+	(wire
+		(pts
 			(xy 210.566 55.88) (xy 203.962 55.88)
 		)
@@
 	(wire
 		(pts
-			(xy 171.704 55.88) (xy 176.022 55.88)
+			(xy 171.704 55.88) (xy 173.736 55.88)
 		)
 		(stroke
@@
 	(wire
 		(pts
-			(xy 157.48 55.88) (xy 161.544 55.88)
+			(xy 218.44 34.544) (xy 193.294 34.544)
 		)
 		(stroke
@@
 		)
 	)
+	(label "vEnv"
+		(at 236.982 37.084 0)
+		(effects
+			(font
+				(size 1.27 1.27)
+			)
+			(justify left bottom)
+		)
+	)
 	(label "Vinput"
 		(at 23.622 57.15 0)
@@
 	(symbol
 		(lib_id "Amplifier_Operational:TL074")
-		(at 221.742 44.196 0)
+		(at 226.06 37.084 0)
 		(unit 4)
 		(body_style 1)
@@
 		(fields_autoplaced yes)
 		(property "Reference" "U1"
-			(at 221.742 34.544 0)
+			(at 226.06 27.432 0)
 			(show_name no)
 			(do_not_autoplace no)
@@
 		)
 		(property "Value" "TL074"
-			(at 221.742 37.084 0)
+			(at 226.06 29.972 0)
 			(show_name no)
 			(do_not_autoplace no)
@@
 		)
 		(property "Footprint" ""
-			(at 220.472 41.656 0)
+			(at 224.79 34.544 0)
 			(hide yes)
 			(show_name no)
@@
 		)
 		(property "Datasheet" "http://www.ti.com/lit/ds/symlink/tl071.pdf"
-			(at 223.012 39.116 0)
+			(at 227.33 32.004 0)
 			(hide yes)
 			(show_name no)
@@
 		)
 		(property "Description" "Quad Low-Noise JFET-Input Operational Amplifiers, DIP-14/SOIC-14"
-			(at 221.742 44.196 0)
+			(at 226.06 37.084 0)
 			(hide yes)
 			(show_name no)
@@
 		)
 		(property "Sim.Library" "/Users/hayden/dev/STM32_Projects/CompressorPedal/CompressorSim/tl074-quad.lib"
-			(at 221.742 44.196 0)
+			(at 226.06 37.084 0)
 			(hide yes)
 			(show_name no)
@@
 		)
 		(property "Sim.Name" "TL074c"
-			(at 221.742 44.196 0)
+			(at 226.06 37.084 0)
 			(hide yes)
 			(show_name no)
@@
 		)
 		(property "Sim.Device" "SUBCKT"
-			(at 221.742 44.196 0)
+			(at 226.06 37.084 0)
 			(hide yes)
 			(show_name no)
@@
 		)
 		(property "Sim.Pins" "1=1 2=2 3=3 4=4 5=5 6=6 7=7 8=8 9=9 10=10 11=11 12=12 13=13 14=14"
-			(at 221.742 44.196 0)
+			(at 226.06 37.084 0)
 			(hide yes)
 			(show_name no)
@@
 			)
 		)
-		(property "Value" "47k"
+		(property "Value" "100k"
 			(at 96.52 55.88 90)
 			(show_name no)
@@
 			)
 		)
-		(property "Value" "22k"
+		(property "Value" "10k"
 			(at 59.69 77.7239 0)
 			(show_name no)
