File: CompressorSim/CompressorSim.kicad_sch (KiCad schematic)
At the start: 14 parts, among them U1 TL074

Commit message: compressor simulation
Parts:
- removed C1: 10u, symbol Device:C
- removed D1: D, symbol Simulation_SPICE:D
- removed R1, R2, R3: 100k, symbol Device:R_US
- added D3: D, symbol Simulation_SPICE:D
- added R8: 100k, symbol Device:R_US
- added V4, V5: 9, symbol Simulation_SPICE:VDC
- R4: value 22k -> 82k
- V3: value 15 -> 11.5
Connections:
- net Env: now also U1.5 (+)
- net GND: now also V4.2, V5.2
- net RatioAmp: now also R6.1
- net VG: now also V4.1; no longer U1.1, U1.2 (-)
- net at R6.2, R7.1, U1.13 (-): now also D2.1 (K), R8.2; no longer D2.2 (A)
- net HalfRect: now reaches R7.2
- net HalfRect: now also D3.2 (A)
- net vThresh: now reaches U1.12 (+), V3.1
- net at U1.14: now also D2.2 (A), D3.1 (K); no longer D2.1 (K)
- new net: R8.1, V5.1
- no-connect marks 0 -> 5
Other:
- note added: ".PARAM Ratio = 0.99"
- note added: "Max is 13.5, min is 7.3ish"
- moved on the sheet: D2, R5, R6, R7, U1A, U1C, U1D, V3

Commit message: VCA and current source sim
Parts:
- added Q1: NPN, symbol Simulation_SPICE:NPN
- added Q2, Q3: PNP, symbol Simulation_SPICE:PNP
- added R10, R11: 470, symbol Device:R_US
- added R12: 10k, symbol Device:R_US
- added R13: 4k7, symbol Device:R_US
- added R14: 47k, symbol Device:R_US
- added R15, R16: 1k, symbol Device:R_US
- added R9: 2k2, symbol Device:R_US
- added U2: LM13700, symbol Amplifier_Operational:LM13700
- added V6: VSIN, symbol Simulation_SPICE:VSIN
- V5: value 9 -> 8.5
Connections:
- net +18V: now also R10.2, R11.2, U2.11 (V+)
- net GND: now also R13.2, U2.6 (V-), V6.2
- net HalfRect: now also U1.10 (+)
- net VG: now also R12.2, R15.2, R16.2, R9.1
- net at U1.8: now also Q1.2 (B)
- net at U1.9 (-): now also Q1.3 (E), R9.2
- new net: Q3.3 (E), R11.1
- new net: R12.1, U2.10, U2.12
- new net: Q1.1 (C), Q2.1 (C), Q2.2 (B), Q3.2 (B)
- new net: R15.1, U2.13 (-)
- new net: R14.2, R16.1, U2.14 (+)
- new net: Q2.3 (E), R10.1
- new net Iabc: Q3.1 (C), U2.16
- new net VCAout: R13.1, U2.9
- new net Vin: R14.1, V6.1
- no-connect marks 5 -> 11
Other:
- note added: "V5 = threshold control Max is 13.5, min is 7.3ish"
- note removed: "Max is 13.5, min is 7.3ish"
- moved on the sheet: U1C
