File: Simulations/CompressorSim/CompressorSim.kicad_sch (KiCad schematic)
At the start: 26 parts, among them Q1 NPN, Q2 PNP, Q3 PNP, U1 TL074, U2 LM13700

Commit message: voltage divider values picked
Parts:
- removed V3: 11.5, symbol Simulation_SPICE:VDC
- removed V5: 8.5, symbol Simulation_SPICE:VDC
- added R17: 10k, symbol Device:R_US
- added R18, R22: 22k, symbol Device:R_US
- added R19: 39k, symbol Device:R_US
- added R20: Potentiometer, symbol Simulation_SPICE:Potentiometer
- added R21: 33k, symbol Device:R_US
- R12: value 10k -> 47k
- R13: value 4k7 -> 10k
- R14: value 47k -> 220k
- R9: value 2k2 -> 3k3
Connections:
- net +18V: now also R18.1, R22.1
- net GND: now also R19.1, R21.2
- net vThresh: now also R8.1, R20.2; no longer U1.12 (+)
- net at R4.1, U1.6 (-): now also R17.1; no longer R5.1
- new net: R18.2, R19.2, U1.12 (+)
- new net: R20.3, R22.2
- new net: R20.1, R21.1
- new net: R17.2, R5.1
Other:
- note added: ".PARAM Ratio = 0.5"
- note added: ".PARAM Thresh = 0.375"
- note added: "Vthresh = threshold control Max is 12.5, min is 9.2ish"
- note removed: ".PARAM Ratio = 0.99"
- note removed: "V5 = threshold control Max is 13.5, min is 7.3ish"
- moved on the sheet: D2, D3, R4, R5, R7, R8, U1B, U1D

Commit message: compressor sim upgrades
Parts:
- added C1: 1u, symbol Device:C
- added C2: 100n, symbol Device:C
- added R23: 100k, symbol Device:R_US
- added R24: Potentiometer, symbol Simulation_SPICE:Potentiometer
- added R25, R26: 47k, symbol Device:R_US
- added R27: 10k, symbol Device:R_US
Connections:
- net GND: now also R27.1
- net VCAout: now also R24.2; no longer R13.1, U2.9
- net VG: now also R23.2, R26.1
- net at U1.1: now also C2.1, R25.2
- net at U1.2 (-): now also R25.1, R26.2
- net at U1.3 (+): now also C1.2, R23.1
- new net: R24.1, R27.2
- new net: C2.2, R24.3
- new net BufferOut: C1.1, R13.1, U2.9
- no-connect marks 11 -> 8
Other:
- note added: ".PARAM Gain = 0.001"
- moved on the sheet: U1A, V1, V2, V4

Commit message: analog and power section schematics
Parts:
- removed C2: 100n, symbol Device:C
- removed R27: 10k, symbol Device:R_US
- R23: value 100k -> 22k
Connections:
- net VCAout: now also R25.2, U1.1; no longer R24.2
- net at R24.1: now also R23.1
- net at R24.3: now also C1.2
- new net: R24.2, U1.3 (+)
Other:
- note added: ".PARAM Gain = 0.99"
- note removed: ".PARAM Gain = 0.001"
- moved on the sheet: R23, R24, R25, R26, U1A, U2C, U2D

Commit message: ADC driver dialed in
Parts:
- C1: value 1u -> 100n
Connections:
- net BiasedOut: now reaches C1.2, R24.3
Changed lines of the file:
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@@
 		)
 	)
+	(label "BiasedOut"
+		(at 163.83 137.16 0)
+		(effects
+			(font
+				(size 1.27 1.27)
+			)
+			(justify left bottom)
+		)
+	)
 	(label "Env"
 		(at 26.67 66.04 0)
@@
 			)
 		)
-		(property "Value" "1u"
+		(property "Value" "100n"
 			(at 156.21 132.08 90)
 			(show_name no)
